File: christmas_tree.sch (KiCad schematic (older format))
At the start: 49 parts, among them J1 Conn_01x28_Female, J10 Conn_01x28_Female, J2 Conn_01x16_Female, J3 Conn_01x12_Female, J4 Conn_01x16_Female, J5 Conn_01x12_Female, J6 Conn_01x12_Female, J7 Conn_01x16_Female, J8 Conn_01x12_Female, J9 Conn_01x16_Female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

Commit message: Replace attiny13 with atmega48 for now
Parts:
- removed U3: ATTINY13-20SSU, Housings_SOIC:SOIC-8_3.9x4.9mm_Pitch1.27mm, symbol ATTINY13-20SSU
- added CON1: AVR-ISP-6, AVR-ISP-6, symbol AVR-ISP-6
- added J16: Conn_01x02_Female, symbol Conn_01x02_Female
- added R13: 10k, symbol R
- added U15: ATMEGA48-20PU, DIL28, symbol ATMEGA48-20PU
- gave numbers to parts that had none: 21
Connections:
- net BLANK: now also U15.24 ((PCINT9/ADC1)PC1)
- net GCLK: now also U15.11 ((PCINT21/OC0B/T1)PD5)
- net GND: now also CON1.6, U15.22 (GND), U15.8 (GND)
- net MOSI: now also CON1.4, U15.17 ((PCINT3/OC2/MOSI)PB3)
- net SCLK: now also CON1.3, U15.19 ((PCINT5/SCK)PB5)
- net VCC: now also CON1.2, R13.2, U15.20 (AVCC), U15.21 (AREF), U15.7 (VCC)
- net VPRG: now also U15.25 ((PCINT10/ADC2)PC2)
- net XLAT: now also U15.23 ((PCINT8/ADC0)PC0)
- new net MISO: CON1.1, U15.18 ((PCINT4/MISO)PB4)
- new net MQ3_A: U15.28 ((PCINT13/SCL/ADC5)PC5)
- new net RST: CON1.5, R13.1, U15.1 ((PCINT14/~RESET~)PC6)
- new net RX: J16.1 (Pin_1), U15.2 ((PCINT16/RXD)PD0)
- new net TX: J16.2 (Pin_2), U15.3 ((PCINT17/TXD)PD1)
- no-connect marks 33 -> 45
Other:
- moved on the sheet: BT1
