File: christmas_tree.sch (KiCad schematic (older format))
At the start: 39 parts, among them CON1 AVR-ISP-6, J1 Conn_01x12_Female, J10 Conn_01x04_Female, J11 Conn_01x08_Female, J12 Conn_01x16_Female, J13 Conn_01x12_Female, J14 Conn_01x04_Female, J15 Conn_01x12_Female, J16 Conn_01x03_Male, J17 Conn_01x12_Female, J2 Conn_01x12_Female, J3 Conn_01x16_Female, J4 Conn_01x12_Female, J5 Conn_01x04_Female, J6 Conn_01x08_Female, J7 Conn_01x04_Female, J8 Conn_01x04_Female, J9 Conn_01x08_Female, SW1 1825910-6, SW2 1825910-6, U1 TLC5940PWP, U15 ATMEGA48-20PU, U2 TLC5940PWP, U3 SEN-08880, U4 TLC5940PWP, U5 TLC5940PWP, U6 TLC5940PWP, U8 TLC5940PWP, U9 TLC5940PWP

Commit message: Finish routing and generate gerber files
Parts:
- added S1: EG2201A, EG2201A:SW_EG2201A, symbol EG2201A
- CON1: footprint Connectors_Multicomp:Multicomp_MC9A12-1034_2x05x2.54mm_Straight -> Pin_Headers:Pin_Header_Straight_2x03_Pitch2.54mm
Connections:
- net GND: now also R6.2, U3.5; no longer J1.10 (Pin_10), J1.2 (Pin_2), J1.6 (Pin_6), J10.3 (Pin_3), J11.3 (Pin_3), J11.7 (Pin_7), J12.11 (Pin_11), J12.15 (Pin_15), J12.3 (Pin_3), J12.7 (Pin_7), J13.11 (Pin_11), J13.3 (Pin_3), J13.7 (Pin_7), J14.3 (Pin_3), J15.11 (Pin_11), J15.3 (Pin_3), J15.7 (Pin_7), J17.11 (Pin_11), J17.3 (Pin_3), J17.7 (Pin_7), J2.10 (Pin_10), J2.2 (Pin_2), J2.6 (Pin_6), J3.10 (Pin_10), J3.14 (Pin_14), J3.2 (Pin_2), J3.6 (Pin_6), J4.11 (Pin_11), J4.3 (Pin_3), J4.7 (Pin_7), J5.2 (Pin_2), J6.3 (Pin_3), J6.7 (Pin_7), J7.3 (Pin_3), J8.2 (Pin_2), J9.3 (Pin_3), J9.7 (Pin_7), R6.1
- net MQ3_A: now also R6.1
- net VCC: now also BT1.+, J1.10 (Pin_10), J1.2 (Pin_2), J1.6 (Pin_6), J10.3 (Pin_3), J11.3 (Pin_3), J11.7 (Pin_7), J12.11 (Pin_11), J12.15 (Pin_15), J12.3 (Pin_3), J12.7 (Pin_7), J13.11 (Pin_11), J13.3 (Pin_3), J13.7 (Pin_7), J14.3 (Pin_3), J15.11 (Pin_11), J15.3 (Pin_3), J15.7 (Pin_7), J17.11 (Pin_11), J17.3 (Pin_3), J17.7 (Pin_7), J2.10 (Pin_10), J2.2 (Pin_2), J2.6 (Pin_6), J3.10 (Pin_10), J3.14 (Pin_14), J3.2 (Pin_2), J3.6 (Pin_6), J4.11 (Pin_11), J4.3 (Pin_3), J4.7 (Pin_7), J5.2 (Pin_2), J6.3 (Pin_3), J6.7 (Pin_7), J7.3 (Pin_3), J8.2 (Pin_2), J9.3 (Pin_3), J9.7 (Pin_7), U15.20 (AVCC), U15.21 (AREF), U15.7 (VCC), S1.2, S1.5; no longer U3.1, U3.2, U3.3
- new net: S1.1, S1.4, U3.1, U3.2, U3.3
- no-connect marks 30 -> 32
Other:
- moved on the sheet: J16, R6
