File: _saved_christmas_tree.sch (KiCad schematic (older format))
At the start: 39 parts, among them CON1 AVR-ISP-6, J1 Conn_01x12_Female, J10 Conn_01x04_Female, J11 Conn_01x08_Female, J12 Conn_01x16_Female, J13 Conn_01x12_Female, J14 Conn_01x04_Female, J15 Conn_01x12_Female, J16 Conn_01x03_Male, J17 Conn_01x12_Female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

Commit message: Christmas tree edge cut
Parts:
- CON1: footprint Connectors_Multicomp:Multicomp_MC9A12-1034_2x05x2.54mm_Straight -> Pin_Headers:Pin_Header_Straight_2x03_Pitch2.54mm
Changed lines of the file:
@@
 F 0 "CON1" H 5245 1540 50  0000 C CNN
 F 1 "AVR-ISP-6" H 5085 1070 50  0000 L BNN
-F 2 "Connectors_Multicomp:Multicomp_MC9A12-1034_2x05x2.54mm_Straight" V 4830 1340 50  0001 C CNN
+F 2 "Pin_Headers:Pin_Header_Straight_2x03_Pitch2.54mm" V 4830 1340 50  0001 C CNN
 F 3 "" H 5325 1300 50  0001 C CNN
 	1    5350 1300
